Commit message: update

File: urdf/example.urdf (robot description, URDF)
Before this commit: robot simple_arm, 11 links, 10 joints
Links:
- link link_4: geometry collision cylinder length=0.1 radius=0.05; visual cylinder length=0.1 radius=0.05
- link link_5: geometry collision cylinder length=0.1 radius=0.05; visual cylinder length=0.1 radius=0.05
Joints:
- joint joint2: limit lower=0 upper=3.14 effort=5 velocity=2.0 -> lower=-3.10 upper=3.10 effort=5 velocity=2.0
- joint joint3: limit lower=0 upper=2.13 effort=5 velocity=2.0 -> lower=-2.13 upper=2.13 effort=5 velocity=2.0
- joint joint4: limit lower=0 upper=2.65 effort=5 velocity=2.0 -> lower=-2.65 upper=2.65 effort=5 velocity=2.0
- joint joint5: limit lower=0 upper=3.14 effort=5 velocity=2.0 -> lower=-3.10 upper=3.10 effort=5 velocity=2.0
- joint joint6: limit lower=0 upper=2.65 effort=5 velocity=2.0 -> lower=-2.65 upper=2.65 effort=5 velocity=2.0
- joint joint7: limit lower=0 upper=3.14 effort=5 velocity=2.0 -> lower=-3.10 upper=3.10 effort=5 velocity=2.0
